Commit message: New manipulator and navigation param

File: src/nucobot_simulator/nucobot_description/urdf/nucobot-2/nucobot.urdf.xacro (robot description, xacro)
@@ -34,11 +34,11 @@
     <visual>
       <geometry>
-        <box size="0.4 0.02 0.02"/>
-      </geometry>
-      <origin xyz="0 0 0" rpy="0 0 0"/>
-    </visual>
-    <collision>
-      <geometry>
-        <box size="0.4 0.02 0.02"/>
+        <box size="0.2 0.02 0.02"/>
+      </geometry>
+      <origin xyz="0 0 0" rpy="0 0 0"/>
+    </visual>
+    <collision>
+      <geometry>
+        <box size="0.2 0.02 0.02"/>
       </geometry>
       <origin xyz="0 0 0" rpy="0 0 0"/>
@@ -46,5 +46,5 @@
     <inertial>
       <origin xyz="0 0 0"/>
-      <mass value="0.4"/>
+      <mass value="0.2"/>
       <inertia ixx="0.019995" ixy="0.0" ixz="0.0"
                iyy="0.019995" iyz="0.0"
@@ -55,11 +55,11 @@
     <visual>
       <geometry>
-        <box size="0.4 0.02 0.02"/>
-      </geometry>
-      <origin xyz="0 0 0" rpy="0 0 0"/>
-    </visual>
-    <collision>
-      <geometry>
-        <box size="0.4 0.02 0.02"/>
+        <box size="0.2 0.02 0.02"/>
+      </geometry>
+      <origin xyz="0 0 0" rpy="0 0 0"/>
+    </visual>
+    <collision>
+      <geometry>
+        <box size="0.2 0.02 0.02"/>
       </geometry>
       <origin xyz="0 0 0" rpy="0 0 0"/>
@@ -67,5 +67,5 @@
     <inertial>
       <origin xyz="0 0 0"/>
-      <mass value="0.4"/>
+      <mass value="0.2"/>
       <inertia ixx="0.019995" ixy="0.0" ixz="0.0"
                iyy="0.019995" iyz="0.0"
